File: HW2/HW2/pic_circuit.sch (EAGLE design)
At the start: 12 parts, among them J1 USB-MB-H

Commit message: completed schematic
Parts:
- added C5, C6: 0.1uF, pic_circuit:C-US025-025X050
- added MCLR, USER: PUSH, pic_circuit:PUSH
- added R3, R4: 10k, pic_circuit:R-US_0207/10
- added U$4: PICKIT3, pic_circuit:PICKIT3
- added U$5: SLIDE, pic_circuit:SLIDE
- added U$6, U$7: CONN_08, pic_circuit:CONN_08
- C1, C4: value (none) -> 0.1uF
- C2, C3: value (none) -> 10uF
- LED1: value (none) -> RED
- LED2: value (none) -> GREEN
- R1, R2: value (none) -> 330
- U$3: value SLIDE-SWITCH -> OSC; device pic_circuit:SLIDE-SWITCH -> pic_circuit:OSC
Connections:
- removed net N$2: C1.1, U$2.2.VIN, U$3.1
- new net +3V3: C2.+, C4.1, C5.1, C6.1, LED1.A, R3.2, R4.2, U$1.13.VDD, U$1.23.VUSB3V3, U$1.28.AVDD, U$2.3.VOUT, U$4.2.VDD, U$7.2
- new net +5V: C1.1, U$1.15.VBUS, U$2.2.VIN, U$5.1, U$6.2
- new net A0: U$1.2.A0, U$6.8
- new net A1: U$1.3.A1, U$6.7
- new net B13: U$1.24.B13, U$7.6
- new net B14: U$1.25.B14, U$7.7
- new net B15: U$1.26.B15, U$7.8
- new net B2: U$1.6.B2, U$6.6
- new net B3: U$1.7.B3, U$6.5
- new net B7: U$1.16.B7, U$7.3
- new net B8: U$1.17.B8, U$7.4
- new net B9: U$1.18.B9, U$7.5
- new net D+: J1.D+, U$1.21.B10/D+
- new net D-: J1.D-, U$1.22.B11/D-
- new net LED2: LED2.A, U$1.12.A4/LED, U$6.3
- new net MCLR: MCLR.2, R4.1, U$1.1.MCLR, U$4.1.MCLR
- new net N$5: U$1.5.B1/PGC, U$4.5.PGC
- new net N$6: C3.+, U$1.20.VCAP
- new net N$7: U$1.9.A2/OSC1, U$3.1.OSC1
- new net N$8: U$1.10.A3/OSC2, U$3.3.OSC2
- new net N$9: LED2.C, R1.2
- new net USBID: J1.ID, U$1.14.B5/USBID
- new net USER: R3.1, U$1.11.B4/USER, U$6.4, USER.2
- net GND: now also C3.-, C5.2, C6.2, J1.GND, MCLR.1, R1.1, U$1.19.VSS, U$1.27.AVSS, U$1.8.VSS, U$3.2.GND, U$4.3.VSS, U$6.1, U$7.1, USER.1
- net N$1: now also U$5.2; no longer U$3.2
- net N$3: now also U$1.4.B0/PGD, U$4.4.PGD; no longer C2.+, C4.1, LED1.A, U$2.3.VOUT
Other:
- moved on the sheet: C1, C2, C3, C4, J1, LED1, LED2, R1, R2, U$2
