File: HW2/pic_circuit.sch (EAGLE design)
At the start: 22 parts, among them J1 USB-MB-H

Commit message: completed pub design
Parts:
- LED2: value GREEN -> GRN
- U$1: value PIC32MX250F128B -> PIC32
Changed lines of the file:
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@@
 <setting verticaltext="up"/>
 </settings>
-<grid distance="0.1" unitdist="inch" unit="inch" style="lines" multiple="1" display="yes" altdistance="0.01" altunitdist="inch" altunit="inch"/>
+<grid distance="0.1" unitdist="inch" unit="inch" style="lines" multiple="1" display="no" altdistance="0.01" altunitdist="inch" altunit="inch"/>
 <layers>
 <layer number="1" name="Top" color="4" fill="1" visible="no" active="no"/>
@@
 </classes>
 <parts>
-<part name="U$1" library="pic_circuit" deviceset="PIC32MX250F128B" device=""/>
+<part name="U$1" library="pic_circuit" deviceset="PIC32MX250F128B" device="" value="PIC32"/>
 <part name="J1" library="pic_circuit" deviceset="USB" device="-MB-H"/>
-<part name="U$2" library="pic_circuit" deviceset="MCP1702" device=""/>
 <part name="C1" library="pic_circuit" deviceset="C-US" device="025-025X050" value="0.1uF"/>
 <part name="R1" library="pic_circuit" deviceset="R-US_" device="0207/10" value="330"/>
@@
 <part name="C4" library="pic_circuit" deviceset="C-US" device="025-025X050" value="0.1uF"/>
 <part name="LED1" library="pic_circuit" deviceset="LED" device="3MM" value="RED"/>
-<part name="LED2" library="pic_circuit" deviceset="LED" device="3MM" value="GREEN"/>
+<part name="LED2" library="pic_circuit" deviceset="LED" device="3MM" value="GRN"/>
 <part name="R2" library="pic_circuit" deviceset="R-US_" device="0207/10" value="330"/>
 <part name="GND2" library="pic_circuit" deviceset="GND" device=""/>
@@
 <part name="+3V3" library="pic_circuit" deviceset="+3V3" device=""/>
 <part name="GND3" library="pic_circuit" deviceset="GND" device=""/>
-<part name="U$5" library="pic_circuit" deviceset="SLIDE" device=""/>
 <part name="GND4" library="pic_circuit" deviceset="GND" device=""/>
 <part name="P+3" library="pic_circuit" deviceset="+5V" device=""/>
@@
 <part name="P+1" library="pic_circuit" deviceset="+5V" device=""/>
 <part name="+3V8" library="pic_circuit" deviceset="+3V3" device=""/>
+<part name="U$2" library="pic_circuit" deviceset="MCP1702" device=""/>
+<part name="U$5" library="pic_circuit" deviceset="SLIDE" device=""/>
 </parts>
 <sheets>
@@
 <instance part="U$1" gate="G$1" x="0" y="0"/>
 <instance part="J1" gate="G$1" x="-60.96" y="-55.88" rot="R180"/>
-<instance part="U$2" gate="G$1" x="0" y="-55.88"/>
 <instance part="C1" gate="G$1" x="-22.86" y="-60.96"/>
 <instance part="R1" gate="G$1" x="63.5" y="-73.66" rot="R90"/>
@@
 <instance part="+3V3" gate="G$1" x="-40.64" y="27.94" rot="R270"/>
 <instance part="GND3" gate="1" x="-40.64" y="20.32"/>
-<instance part="U$5" gate="G$1" x="-40.64" y="-58.42"/>
 <instance part="GND4" gate="1" x="38.1" y="-20.32"/>
 <instance part="P+3" gate="1" x="27.94" y="-33.02" rot="R270"/>
@@
 <instance part="P+1" gate="1" x="81.28" y="17.78"/>
 <instance part="+3V8" gate="G$1" x="81.28" y="-12.7"/>
+<instance part="U$2" gate="G$1" x="0" y="-55.88"/>
+<instance part="U$5" gate="G$1" x="-40.64" y="-58.42"/>
 </instances>
 <busses>
@@
 <segment>
 <pinref part="GND1" gate="1" pin="GND"/>
-<pinref part="U$2" gate="G$1" pin="1.GND"/>
 <wire x1="0" y1="-68.58" x2="0" y2="-66.04" width="0.1524" layer="91"/>
 <wire x1="0" y1="-68.58" x2="-22.86" y2="-68.58" width="0.1524" layer="91"/>
@@
 <pinref part="C2" gate="G$1" pin="-"/>
 <wire x1="33.02" y1="-68.58" x2="33.02" y2="-66.04" width="0.1524" layer="91"/>
+<pinref part="U$2" gate="G$1" pin="1.GND"/>
 </segment>
 <segment>
@@
 <net name="+3V3" class="0">
 <segment>
-<pinref part="U$2" gate="G$1" pin="3.VOUT"/>
 <wire x1="17.78" y1="-55.88" x2="22.86" y2="-55.88" width="0.1524" layer="91"/>
 <pinref part="C2" gate="G$1" pin="+"/>
@@
 <wire x1="43.18" y1="-55.88" x2="43.18" y2="-53.34" width="0.1524" layer="91"/>
 <junction x="43.18" y="-55.88"/>
+<pinref part="U$2" gate="G$1" pin="3.VOUT"/>
 </segment>
 <segment>
@@
 <net name="+5V" class="0">
 <segment>
-<pinref part="U$2" gate="G$1" pin="2.VIN"/>
 <wire x1="-33.02" y1="-55.88" x2="-27.94" y2="-55.88" width="0.1524" layer="91"/>
 <pinref part="C1" gate="G$1" pin="1"/>
@@
 <wire x1="-27.94" y1="-53.34" x2="-27.94" y2="-55.88" width="0.1524" layer="91"/>
 <junction x="-27.94" y="-55.88"/>
+<pinref part="U$2" gate="G$1" pin="2.VIN"/>
 <pinref part="U$5" gate="G$1" pin="1"/>
 </segment>

Commit message: created hw 3 folder
Connections:
- net +3V3: now also U$6.2; no longer U$7.2
- net +5V: now also U$7.2; no longer U$6.2
Changed lines of the file:
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@@
 <part name="GND12" library="pic_circuit" deviceset="GND" device=""/>
 <part name="GND13" library="pic_circuit" deviceset="GND" device=""/>
+<part name="U$2" library="pic_circuit" deviceset="MCP1702" device=""/>
+<part name="U$5" library="pic_circuit" deviceset="SLIDE" device=""/>
 <part name="P+1" library="pic_circuit" deviceset="+5V" device=""/>
 <part name="+3V8" library="pic_circuit" deviceset="+3V3" device=""/>
-<part name="U$2" library="pic_circuit" deviceset="MCP1702" device=""/>
-<part name="U$5" library="pic_circuit" deviceset="SLIDE" device=""/>
 </parts>
 <sheets>
@@
 <instance part="GND12" gate="1" x="73.66" y="-20.32"/>
 <instance part="GND13" gate="1" x="73.66" y="10.16"/>
-<instance part="P+1" gate="1" x="81.28" y="17.78"/>
-<instance part="+3V8" gate="G$1" x="81.28" y="-12.7"/>
 <instance part="U$2" gate="G$1" x="0" y="-55.88"/>
 <instance part="U$5" gate="G$1" x="-40.64" y="-58.42"/>
+<instance part="P+1" gate="1" x="81.28" y="-12.7"/>
+<instance part="+3V8" gate="G$1" x="81.28" y="17.78"/>
 </instances>
 <busses>
@@
 </segment>
 <segment>
-<pinref part="U$7" gate="G$1" pin="2"/>
-<wire x1="68.58" y1="-15.24" x2="81.28" y2="-15.24" width="0.1524" layer="91"/>
+<pinref part="U$6" gate="G$1" pin="2"/>
+<wire x1="68.58" y1="15.24" x2="81.28" y2="15.24" width="0.1524" layer="91"/>
 <pinref part="+3V8" gate="G$1" pin="+3V3"/>
 </segment>
@@
 </segment>
 <segment>
-<pinref part="U$6" gate="G$1" pin="2"/>
-<wire x1="68.58" y1="15.24" x2="81.28" y2="15.24" width="0.1524" layer="91"/>
+<pinref part="U$7" gate="G$1" pin="2"/>
+<wire x1="68.58" y1="-15.24" x2="81.28" y2="-15.24" width="0.1524" layer="91"/>
 <pinref part="P+1" gate="1" pin="+5V"/>
 </segment>
